Commit message: add active gripper groups + open/closed targets

File: baxter/baxter_moveit_config/config/baxter_base.srdf.xacro (robot description, xacro)
@@ -25,7 +25,15 @@
     <group name="left_hand">
         <chain base_link="left_hand" tip_link="$(arg left_tip_name)" />
+        <joint name="l_gripper_l_finger_joint" />
+        <joint name="l_gripper_r_finger_joint" />
+        <link name="l_gripper_l_finger_tip" />
+        <link name="l_gripper_r_finger_tip" />
     </group>
     <group name="right_hand">
         <chain base_link="right_hand" tip_link="$(arg right_tip_name)" />
+        <joint name="r_gripper_l_finger_joint" />
+        <joint name="r_gripper_r_finger_joint" />
+        <link name="r_gripper_l_finger_tip" />
+        <link name="r_gripper_r_finger_tip" />
     </group>
     <!--END EFFECTOR: Purpose: Represent information about an end effector.-->
@@ -50,4 +58,20 @@
         <joint name="right_w1" value="1.26" />
         <joint name="right_w2" value="0" />
+    </group_state>
+    <group_state name="closed" group="right_hand">
+        <joint name="r_gripper_l_finger_joint" value="0.0" />
+        <joint name="r_gripper_r_finger_joint" value="0.0" />
+    </group_state>
+    <group_state name="open" group="right_hand">
+        <joint name="r_gripper_l_finger_joint" value="0.020833" />
+        <joint name="r_gripper_r_finger_joint" value="-0.020833" />
+    </group_state>
+    <group_state name="closed" group="left_hand">
+        <joint name="l_gripper_l_finger_joint" value="0.0" />
+        <joint name="l_gripper_r_finger_joint" value="0.0" />
+    </group_state>
+    <group_state name="open" group="left_hand">
+        <joint name="l_gripper_l_finger_joint" value="0.020833" />
+        <joint name="l_gripper_r_finger_joint" value="-0.020833" />
     </group_state>
     <!--END EFFECTOR: Purpose: Represent information about an end effector.-->
